File: Modularized/HT-Chorus/HT-Chorus.kicad_pcb (KiCad board)
At the start: 4 copper layers, 57 parts, among them Q1 2SC1740?, T1 2SC1740, T2 2SC1740, T3 2SC1740, U1 MN3207, U2 MN3102

Commit message: save point
Parts:
- added INPUT: REF**, MyKi_TH_Board_Features:Labled-Circle, F.Cu at (119.4, 106.7)
- added LFO: REF**, MyKi_TH_Board_Features:Labled-Circle, F.Cu at (35.6, 127.0)
- added OUTPUT: REF**, MyKi_TH_Board_Features:Labled-Circle, F.Cu at (132.1, 132.1)
- added VE: REF**, MyKi_TH_Board_Features:Labled-Circle, F.Cu at (128.3, 97.8)
Routing:
- net /Input: track 22.9 -> 7.62 mm
- net /LFO: track 10.2 -> 2.54 mm
- net VE: vias 8 -> 9
Other:
- board text added: "HT-Chorus"
Changed lines of the file:
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@@
   (general
     (thickness 1.6)
-    (drawings 0)
-    (tracks 507)
+    (drawings 1)
+    (tracks 506)
     (zones 0)
-    (modules 57)
+    (modules 61)
     (nets 38)
   )
@@
     (add_net VE)
   )
+  (module MyKi_TH_Board_Features:Labled-Circle (layer F.Cu)
+    (at 35.56 127)
+    (tags "label labeled circle node ")
+    (attr virtual)
+    (fp_text reference LFO (at 0 1.905) (layer F.Adhes)
+      (effects (font (size 1 1) (thickness 0.25)))
+    )
+    (fp_text value REF** (at 0 -2.54 180) (layer F.SilkS) hide
+      (effects (font (size 1 1) (thickness 0.15)))
+    )
+    (fp_circle (center 0 0) (end 0.762 0.508) (layer F.Adhes) (width 0.4))
+  )
+  (module MyKi_TH_Board_Features:Labled-Circle (layer F.Cu)
+    (at 132.08 132.08)
+    (tags "label labeled circle node ")
+    (attr virtual)
+    (fp_text reference OUTPUT (at 0 1.905) (layer F.Adhes)
+      (effects (font (size 1 1) (thickness 0.25)))
+    )
+    (fp_text value REF** (at 0 -2.54 180) (layer F.SilkS) hide
+      (effects (font (size 1 1) (thickness 0.15)))
+    )
+    (fp_circle (center 0 0) (end 0.762 0.508) (layer F.Adhes) (width 0.4))
+  )
+  (module MyKi_TH_Board_Features:Labled-Circle (layer F.Cu)
+    (at 128.27 97.79 180)
+    (tags "label labeled circle node ")
+    (attr virtual)
+    (fp_text reference VE (at 0 1.905 180) (layer F.Adhes)
+      (effects (font (size 1 1) (thickness 0.25)))
+    )
+    (fp_text value REF** (at 0 -2.54) (layer F.SilkS) hide
+      (effects (font (size 1 1) (thickness 0.15)))
+    )
+    (fp_circle (center 0 0) (end 0.762 0.508) (layer F.Adhes) (width 0.4))
+  )
+  (module MyKi_TH_Board_Features:Labled-Circle (layer F.Cu)
+    (at 119.38 106.68 180)
+    (tags "label labeled circle node ")
+    (attr virtual)
+    (fp_text reference INPUT (at 0 1.905 180) (layer F.Adhes)
+      (effects (font (size 1 1) (thickness 0.25)))
+    )
+    (fp_text value REF** (at 0 -2.54) (layer F.SilkS) hide
+      (effects (font (size 1 1) (thickness 0.15)))
+    )
+    (fp_circle (center 0 0) (end 0.762 0.508) (layer F.Adhes) (width 0.4))
+  )
   (module MyKi_Generics:200Mil_2TH_Polar_Generic placed (layer F.Cu)
     (at 63.5 119.38 270)
@@
       (net 15 "Net-(C11-Pad1)") (zone_connect 2))
   )
+  (gr_text HT-Chorus (at 115.57 118.11) (layer B.CrtYd)
+    (effects (font (size 1.5 1.5) (thickness 0.3)))
+  )
+  (via (at 128.27 97.79) (size 1.5) (drill 0.8) (layers F.Cu B.Cu) (net 37))
   (segment (start 119.38 106.68) (end 119.38 111.76) (width 0.5) (layer B.Cu) (net 1))
   (segment (start 45.72 124.46) (end 45.72 134.62) (width 0.5) (layer B.Cu) (net 3))
@@
   (segment (start 175.895 105.41) (end 175.895 118.11) (width 0.5) (layer F.Cu) (net 37))
   (segment (start 175.26 101.6) (end 175.895 105.41) (width 0.5) (layer F.Cu) (net 37))
-  (segment (start 119.38 106.68) (end 119.38 91.44) (width 0.5) (layer In2.Cu) (net 1))
   (via (at 119.38 106.68) (size 1.5) (drill 0.8) (layers F.Cu B.Cu) (net 1))
   (segment (start 119.38 111.76) (end 119.38 114.3) (width 0.5) (layer B.Cu) (net 1) (status C00000))
@@
   (segment (start 35.56 124.46) (end 35.56 127) (width 0.5) (layer B.Cu) (net 25) (status 400000))
   (via (at 35.56 127) (size 1.5) (drill 0.8) (layers F.Cu B.Cu) (net 25))
-  (segment (start 35.56 127) (end 27.94 127) (width 0.5) (layer F.Cu) (net 25))
   (segment (start 45.720001 111.76) (end 45.72 109.22) (width 0.5) (layer B.Cu) (net 26) (status C00000))
   (segment (start 45.72 116.84) (end 45.72 114.3) (width 0.5) (layer B.Cu) (net 26))
