File: Modularized/HT-Final/HT-Final.kicad_pcb (KiCad board)
At the start: 2 copper layers, 65 parts, among them T8 2SC1740?

Commit message: save point
Parts:
- added CH0: REF**, MyKi_TH_Board_Features:Labled-Circle, F.Cu at (203.2, 68.6)
- added CH1: REF**, MyKi_TH_Board_Features:Labled-Circle, F.Cu at (198.1, 40.6)
- added LVCF(M): REF**, MyKi_TH_Board_Features:Labled-Circle, F.Cu at (170.2, 40.6)
- added PERC9: REF**, MyKi_TH_Board_Features:Labled-Circle, F.Cu at (104.1, 40.6)
- added UVCF(M): REF**, MyKi_TH_Board_Features:Labled-Circle, F.Cu at (210.8, 40.6)
- added VE: REF**, MyKi_TH_Board_Features:Labled-Circle, F.Cu at (238.8, 40.6)
Routing:
- net VE: track 59.3 -> 67.0 mm, vias 4 -> 5
- net Net-(C27-Pad1): track 30.5 -> 31.1 mm
Other:
- board text added: "HT-FINAL"
Changed lines of the file:
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@@
   (general
     (thickness 1.6)
-    (drawings 2)
-    (tracks 450)
+    (drawings 3)
+    (tracks 454)
     (zones 0)
-    (modules 65)
+    (modules 71)
     (nets 51)
   )
@@
     (add_net VE)
   )
+  (module MyKi_TH_Board_Features:Labled-Circle (layer F.Cu)
+    (at 238.76 40.64)
+    (tags "label labeled circle node ")
+    (attr virtual)
+    (fp_text reference VE (at 0 -1.905) (layer F.Adhes)
+      (effects (font (size 1 1) (thickness 0.25)))
+    )
+    (fp_text value REF** (at 0 -2.54 180) (layer F.SilkS) hide
+      (effects (font (size 1 1) (thickness 0.15)))
+    )
+    (fp_circle (center 0 0) (end 0.762 0.508) (layer F.Adhes) (width 0.4))
+  )
+  (module MyKi_TH_Board_Features:Labled-Circle (layer F.Cu)
+    (at 210.82 40.64)
+    (tags "label labeled circle node ")
+    (attr virtual)
+    (fp_text reference "UVCF(M)" (at 0 -1.905) (layer F.Adhes)
+      (effects (font (size 1 1) (thickness 0.25)))
+    )
+    (fp_text value REF** (at 0 -2.54 180) (layer F.SilkS) hide
+      (effects (font (size 1 1) (thickness 0.15)))
+    )
+    (fp_circle (center 0 0) (end 0.762 0.508) (layer F.Adhes) (width 0.4))
+  )
+  (module MyKi_TH_Board_Features:Labled-Circle (layer F.Cu)
+    (at 203.2 68.58)
+    (tags "label labeled circle node ")
+    (attr virtual)
+    (fp_text reference CH0 (at 0 1.905) (layer F.Adhes)
+      (effects (font (size 1 1) (thickness 0.25)))
+    )
+    (fp_text value REF** (at 0 -2.54 180) (layer F.SilkS) hide
+      (effects (font (size 1 1) (thickness 0.15)))
+    )
+    (fp_circle (center 0 0) (end 0.762 0.508) (layer F.Adhes) (width 0.4))
+  )
+  (module MyKi_TH_Board_Features:Labled-Circle (layer F.Cu)
+    (at 198.12 40.64)
+    (tags "label labeled circle node ")
+    (attr virtual)
+    (fp_text reference CH1 (at 0 -1.905) (layer F.Adhes)
+      (effects (font (size 1 1) (thickness 0.25)))
+    )
+    (fp_text value REF** (at 0 -2.54 180) (layer F.SilkS) hide
+      (effects (font (size 1 1) (thickness 0.15)))
+    )
+    (fp_circle (center 0 0) (end 0.762 0.508) (layer F.Adhes) (width 0.4))
+  )
   (module MyKi_TH_Board_Features:breadboard-endless (layer F.Cu)
     (at 228.6 53.34)
@@
     )
   )
+  (module MyKi_TH_Board_Features:Labled-Circle (layer F.Cu)
+    (at 104.14 40.64)
+    (tags "label labeled circle node ")
+    (attr virtual)
+    (fp_text reference PERC9 (at 0 -1.905) (layer F.Adhes)
+      (effects (font (size 1 1) (thickness 0.25)))
+    )
+    (fp_text value REF** (at 0 -2.54 180) (layer F.SilkS) hide
+      (effects (font (size 1 1) (thickness 0.15)))
+    )
+    (fp_circle (center 0 0) (end 0.762 0.508) (layer F.Adhes) (width 0.4))
+  )
+  (module MyKi_TH_Board_Features:Labled-Circle (layer F.Cu)
+    (at 170.18 40.64)
+    (tags "label labeled circle node ")
+    (attr virtual)
+    (fp_text reference "LVCF(M)" (at 0 -1.905) (layer F.Adhes)
+      (effects (font (size 1 1) (thickness 0.25)))
+    )
+    (fp_text value REF** (at 0 -2.54 180) (layer F.SilkS) hide
+      (effects (font (size 1 1) (thickness 0.15)))
+    )
+    (fp_circle (center 0 0) (end 0.762 0.508) (layer F.Adhes) (width 0.4))
+  )
+  (gr_text HT-FINAL (at 184.15 38.1) (layer F.SilkS)
+    (effects (font (size 1.5 1.5) (thickness 0.3)))
+  )
   (gr_text "Rhythm Vol" (at 134.62 71.12) (layer F.CrtYd)
     (effects (font (size 0.8 0.8) (thickness 0.2)))
@@
   (segment (start 243.84 60.96) (end 243.84 58.42) (width 0.5) (layer F.Cu) (net 24) (status 400000))
   (via (at 243.84 58.42) (size 1.5) (drill 0.8) (layers F.Cu B.Cu) (net 24))
+  (segment (start 238.76 48.26) (end 238.76 40.64) (width 0.5) (layer B.Cu) (net 33))
+  (via (at 238.76 40.64) (size 1.5) (drill 0.8) (layers F.Cu B.Cu) (net 33))
   (segment (start 104.14 48.26) (end 104.14 40.64) (width 0.5) (layer B.Cu) (net 37))
   (via (at 104.14 40.64) (size 1.5) (drill 0.8) (layers F.Cu B.Cu) (net 37))
@@
   (segment (start 261.62 60.96) (end 261.62 68.58) (width 0.5) (layer B.Cu) (net 44))
   (via (at 261.62 68.58) (size 1.5) (drill 0.8) (layers F.Cu B.Cu) (net 44))
+  (segment (start 243.84 39.37) (end 236.22 39.37) (width 0.5) (layer F.Cu) (net 47))
+  (segment (start 243.84 39.37) (end 246.38 40.64) (width 0.5) (layer F.Cu) (net 47))
+  (segment (start 233.670266 45.492295) (end 233.670266 40.649734) (width 0.5) (layer B.Cu) (net 47))
+  (segment (start 233.670266 40.649734) (end 233.68 40.64) (width 0.5) (layer B.Cu) (net 47))
+  (via (at 233.68 40.64) (size 1.5) (drill 0.8) (layers F.Cu B.Cu) (net 47))
+  (segment (start 246.38 45.72) (end 246.38 48.26) (width 0.5) (layer B.Cu) (net 47) (status 800000))
+  (via (at 246.38 40.64) (size 1.5) (drill 0.8) (layers F.Cu B.Cu) (net 47))
+  (segment (start 246.38 43.18) (end 246.38 40.64) (width 0.5) (layer B.Cu) (net 47))
+  (segment (start 246.38 45.72) (end 246.38 43.18) (width 0.5) (layer B.Cu) (net 47))
+  (segment (start 233.68 40.64) (end 236.22 39.37) (width 0.5) (layer F.Cu) (net 47))
   (segment (start 210.82 43.18) (end 218.44 43.18) (width 0.5) (layer F.Cu) (net 50))
   (segment (start 218.44 43.18) (end 220.98 40.64) (width 0.5) (layer F.Cu) (net 50))
@@
   (via (at 220.98 40.64) (size 1.5) (drill 0.8) (layers F.Cu B.Cu) (net 50))
   (via (at 208.28 40.64) (size 1.5) (drill 0.8) (layers F.Cu B.Cu) (net 50))
-  (segment (start 233.68 40.64) (end 246.38 40.64) (width 0.5) (layer F.Cu) (net 47))
-  (segment (start 233.670266 45.492295) (end 233.670266 40.649734) (width 0.5) (layer B.Cu) (net 47))
-  (segment (start 233.670266 40.649734) (end 233.68 40.64) (width 0.5) (layer B.Cu) (net 47))
-  (via (at 233.68 40.64) (size 1.5) (drill 0.8) (layers F.Cu B.Cu) (net 47))
   (segment (start 256.54 68.58) (end 243.84 68.58) (width 0.5) (layer F.Cu) (net 33))
   (segment (start 256.54 66.04) (end 256.54 68.58) (width 0.5) (layer B.Cu) (net 33))
@@
   (segment (start 233.68 50.8) (end 233.68 48.04203) (width 0.5) (layer B.Cu) (net 47))
   (segment (start 233.68 48.04203) (end 233.670266 48.032296) (width 0.5) (layer B.Cu) (net 47))
-  (segment (start 246.38 48.26) (end 246.38 45.72) (width 0.5) (layer B.Cu) (net 47) (status 400000))
-  (via (at 246.38 40.64) (size 1.5) (drill 0.8) (layers F.Cu B.Cu) (net 47))
-  (segment (start 246.38 43.18) (end 246.38 40.64) (width 0.5) (layer B.Cu) (net 47))
-  (segment (start 246.38 45.72) (end 246.38 43.18) (width 0.5) (layer B.Cu) (net 47))
   (segment (start 241.3 45.72) (end 236.22 45.72) (width 0.5) (layer F.Cu) (net 26))
   (via (at 236.22 45.72) (size 1.5) (drill 0.8) (layers F.Cu B.Cu) (net 26))
