File: Modularized/HT-Mutes/HT-Mutes.sch (KiCad schematic (older format))
At the start: 21 parts, among them Q1 2SJ104?, Q2 2SJ104, U1 LA6358?

Commit message: save point
Parts:
- C1, C2, D1, D2, D3, D4: footprint (none) -> MyKi_Generics:200Mil_2TH_Polar_Generic
- Q1: footprint (none) -> TO_SOT_Packages_THT:TO-92_Inline_Narrow_Oval
- Q2: value 2SJ104 -> 2SJ104?; footprint (none) -> TO_SOT_Packages_THT:TO-92_Inline_Narrow_Oval
- R1, R10, R11, R12, R2, R3, R4, R5, R6, R7, R8, R9: footprint (none) -> MyKi_Generics:200Mil_2TH_Generic
- U1: footprint (none) -> MyKi_TH_IC:300Mil_DIP14
