File: Modularized/HT-VCF-Pre/HT-VCF-Pre.kicad_pcb (KiCad board)
At the start: 2 copper layers, 28 parts, among them J1 DB25_Female

Commit message: save point
Parts:
- added LOSC: REF**, MyKi_TH_Board_Features:Labled-Circle, F.Cu at (106.7, 91.4)
- added UOSC: REF**, MyKi_TH_Board_Features:Labled-Circle, F.Cu at (68.6, 114.3)
- added VBC: REF**, MyKi_TH_Board_Features:Labled-Circle, F.Cu at (73.7, 116.8)
Routing:
- net VBC: track 164.9 -> 152.7 mm, vias 8 -> 9
- net /LOSC: track 7.62 -> 15.2 mm, vias 2 -> 3
- net (no net): track 0.00 -> 7.62 mm, vias 0 -> 2
- net /UOSC: track 2.54 -> 5.08 mm, vias 0 -> 1
- net Net-(C7-Pad1): track 47.7 -> 46.8 mm
Other:
- board text added: "HT-VCF-Pre"
Changed lines of the file:
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@@
   (general
     (thickness 1.6)
-    (drawings 0)
-    (tracks 344)
+    (drawings 1)
+    (tracks 347)
     (zones 0)
-    (modules 28)
+    (modules 31)
     (nets 45)
   )
@@
     (add_net "Net-(TC4066-1-Pad5)")
     (add_net VBC)
+  )
+  (module MyKi_TH_Board_Features:Labled-Circle (layer F.Cu)
+    (at 73.66 116.84)
+    (tags "label labeled circle node ")
+    (attr virtual)
+    (fp_text reference VBC (at 0 -2.032) (layer F.Adhes)
+      (effects (font (size 1 1) (thickness 0.25)))
+    )
+    (fp_text value REF** (at 0 -2.54 180) (layer F.SilkS) hide
+      (effects (font (size 1 1) (thickness 0.15)))
+    )
+    (fp_circle (center 0 0) (end 0.762 0.508) (layer F.Adhes) (width 0.4))
+  )
+  (module MyKi_TH_Board_Features:Labled-Circle (layer F.Cu)
+    (at 106.68 91.44)
+    (tags "label labeled circle node ")
+    (attr virtual)
+    (fp_text reference LOSC (at 0 2.032) (layer F.Adhes)
+      (effects (font (size 1 1) (thickness 0.25)))
+    )
+    (fp_text value REF** (at 0 -2.54 180) (layer F.SilkS) hide
+      (effects (font (size 1 1) (thickness 0.15)))
+    )
+    (fp_circle (center 0 0) (end 0.762 0.508) (layer F.Adhes) (width 0.4))
   )
   (module MyKi_Generics:200Mil_2TH_Generic placed (layer F.Cu)
@@
     (fp_arc (start -43.18 0) (end -43.18 0.635) (angle 90) (layer B.SilkS) (width 0.15))
   )
+  (module MyKi_TH_Board_Features:Labled-Circle (layer F.Cu)
+    (at 68.58 114.3)
+    (tags "label labeled circle node ")
+    (attr virtual)
+    (fp_text reference UOSC (at 0 2.032) (layer F.Adhes)
+      (effects (font (size 1 1) (thickness 0.25)))
+    )
+    (fp_text value REF** (at 0 -2.54 180) (layer F.SilkS) hide
+      (effects (font (size 1 1) (thickness 0.15)))
+    )
+    (fp_circle (center 0 0) (end 0.762 0.508) (layer F.Adhes) (width 0.4))
+  )
+  (gr_text HT-VCF-Pre (at 91.948 78.232) (layer F.SilkS)
+    (effects (font (size 1.5 1.5) (thickness 0.3)))
+  )
+  (segment (start 58.42 109.22) (end 58.42 114.3) (width 0.5) (layer B.Cu) (net 0))
+  (segment (start 73.66 111.76) (end 73.66 116.84) (width 0.5) (layer B.Cu) (net 1))
+  (via (at 73.66 116.84) (size 1.5) (drill 0.8) (layers F.Cu B.Cu) (net 1))
+  (via (at 58.42 109.22) (size 1.5) (drill 0.8) (layers F.Cu B.Cu) (net 1))
+  (segment (start 60.96 110.236) (end 58.42 109.22) (width 0.5) (layer F.Cu) (net 1))
+  (segment (start 72.136 110.744) (end 60.96 110.236) (width 0.5) (layer F.Cu) (net 1))
+  (segment (start 73.66 111.76) (end 72.136 110.744) (width 0.5) (layer F.Cu) (net 1))
+  (via (at 73.66 111.76) (size 1.5) (drill 0.8) (layers F.Cu B.Cu) (net 1))
+  (segment (start 73.66 109.22) (end 73.66 111.76) (width 0.5) (layer B.Cu) (net 1) (status 400000))
+  (via (at 58.42 114.3) (size 1.5) (drill 0.8) (layers F.Cu B.Cu) (net 0))
+  (segment (start 58.42 114.3) (end 55.88 114.3) (width 0.5) (layer F.Cu) (net 0))
+  (via (at 55.88 114.3) (size 1.5) (drill 0.8) (layers F.Cu B.Cu) (net 0))
   (segment (start 76.2 96.52) (end 76.2 93.98) (width 0.5) (layer B.Cu) (net 1))
   (segment (start 124.46 96.52) (end 124.46 99.06) (width 0.5) (layer B.Cu) (net 1))
   (via (at 124.46 96.52) (size 1.5) (drill 0.8) (layers F.Cu B.Cu) (net 1))
-  (segment (start 120.015 94.615) (end 124.46 96.52) (width 0.5) (layer F.Cu) (net 1))
-  (segment (start 109.855 92.075) (end 120.015 94.615) (width 0.5) (layer F.Cu) (net 1))
-  (segment (start 106.045 91.44) (end 109.855 92.075) (width 0.5) (layer F.Cu) (net 1))
-  (segment (start 100.965 92.71) (end 106.045 91.44) (width 0.5) (layer F.Cu) (net 1))
+  (segment (start 119.888 95.504) (end 124.46 96.52) (width 0.5) (layer F.Cu) (net 1))
+  (segment (start 110.363 94.107) (end 119.888 95.504) (width 0.5) (layer F.Cu) (net 1))
+  (segment (start 107.188 93.472) (end 110.363 94.107) (width 0.5) (layer F.Cu) (net 1))
+  (segment (start 100.965 92.71) (end 107.188 93.472) (width 0.5) (layer F.Cu) (net 1))
   (segment (start 95.25 93.98) (end 100.965 92.71) (width 0.5) (layer F.Cu) (net 1))
   (segment (start 86.36 94.615) (end 95.25 93.98) (width 0.5) (layer F.Cu) (net 1))
@@
   (segment (start 76.2 101.6) (end 76.2 99.06) (width 0.5) (layer B.Cu) (net 1) (status 400000))
   (via (at 55.88 111.76) (size 1.5) (drill 0.8) (layers F.Cu B.Cu) (net 1))
-  (segment (start 57.785 111.125) (end 55.88 111.76) (width 0.5) (layer F.Cu) (net 1))
-  (segment (start 59.055 109.22) (end 57.785 111.125) (width 0.5) (layer F.Cu) (net 1))
-  (segment (start 59.69 106.68) (end 59.055 109.22) (width 0.5) (layer F.Cu) (net 1))
-  (segment (start 59.69 102.87) (end 59.69 106.68) (width 0.5) (layer F.Cu) (net 1))
+  (segment (start 56.896 110.236) (end 55.88 111.76) (width 0.5) (layer F.Cu) (net 1))
+  (segment (start 56.896 107.696) (end 56.896 110.236) (width 0.5) (layer F.Cu) (net 1))
+  (segment (start 58.166 104.648) (end 56.896 107.696) (width 0.5) (layer F.Cu) (net 1))
+  (segment (start 59.69 102.87) (end 58.166 104.648) (width 0.5) (layer F.Cu) (net 1))
   (segment (start 62.865 95.885) (end 59.69 102.87) (width 0.5) (layer F.Cu) (net 1))
   (segment (start 64.77 94.615) (end 62.865 95.885) (width 0.5) (layer F.Cu) (net 1))
@@
   (segment (start 124.46 113.03) (end 125.73 110.49) (width 0.5) (layer F.Cu) (net 1))
   (segment (start 124.46 99.06) (end 124.46 101.6) (width 0.5) (layer B.Cu) (net 1) (status 800000))
-  (segment (start 73.66 109.22) (end 73.66 111.76) (width 0.5) (layer B.Cu) (net 1) (status 400000))
-  (segment (start 73.66 111.76) (end 73.66 114.3) (width 0.5) (layer B.Cu) (net 1))
-  (segment (start 73.66 114.3) (end 73.66 116.84) (width 0.5) (layer B.Cu) (net 1))
-  (segment (start 73.66 116.84) (end 73.66 119.38) (width 0.5) (layer B.Cu) (net 1))
-  (via (at 73.66 119.38) (size 1.5) (drill 0.8) (layers F.Cu B.Cu) (net 1))
-  (segment (start 73.66 119.38) (end 72.39 121.92) (width 0.5) (layer F.Cu) (net 1))
-  (segment (start 72.39 121.92) (end 69.85 123.19) (width 0.5) (layer F.Cu) (net 1))
-  (segment (start 69.85 123.19) (end 63.5 123.19) (width 0.5) (layer F.Cu) (net 1))
-  (segment (start 63.5 123.19) (end 60.96 120.65) (width 0.5) (layer F.Cu) (net 1))
-  (segment (start 60.96 120.65) (end 59.69 118.11) (width 0.5) (layer F.Cu) (net 1))
-  (segment (start 59.69 118.11) (end 58.42 115.57) (width 0.5) (layer F.Cu) (net 1))
-  (segment (start 58.42 115.57) (end 55.88 114.3) (width 0.5) (layer F.Cu) (net 1))
-  (via (at 55.88 114.3) (size 1.5) (drill 0.8) (layers F.Cu B.Cu) (net 1))
   (segment (start 57.15 82.55) (end 58.42 78.74) (width 0.5) (layer F.Cu) (net 2))
   (via (at 57.15 82.55) (size 1.5) (drill 0.8) (layers F.Cu B.Cu) (net 2))
@@
   (via (at 116.84 111.76) (size 1.5) (drill 0.8) (layers F.Cu B.Cu) (net 12))
   (via (at 104.14 93.98) (size 1.5) (drill 0.8) (layers F.Cu B.Cu) (net 12))
-  (segment (start 104.14 93.98) (end 106.045 93.345) (width 0.5) (layer F.Cu) (net 12))
-  (segment (start 106.045 93.345) (end 108.585 93.98) (width 0.5) (layer F.Cu) (net 12))
-  (segment (start 108.585 93.98) (end 110.49 95.25) (width 0.5) (layer F.Cu) (net 12))
-  (segment (start 110.49 95.25) (end 111.76 97.79) (width 0.5) (layer F.Cu) (net 12))
-  (segment (start 111.76 97.79) (end 113.03 104.14) (width 0.5) (layer F.Cu) (net 12))
+  (segment (start 104.14 93.98) (end 107.061 94.869) (width 0.5) (layer F.Cu) (net 12))
+  (segment (start 107.061 94.869) (end 109.601 95.504) (width 0.5) (layer F.Cu) (net 12))
+  (segment (start 109.601 95.504) (end 110.998 96.774) (width 0.5) (layer F.Cu) (net 12))
+  (segment (start 110.998 96.774) (end 112.268 99.314) (width 0.5) (layer F.Cu) (net 12))
+  (segment (start 112.268 99.314) (end 113.03 104.14) (width 0.5) (layer F.Cu) (net 12))
   (segment (start 113.03 104.14) (end 113.665 106.68) (width 0.5) (layer F.Cu) (net 12))
   (segment (start 113.665 106.68) (end 114.935 109.22) (width 0.5) (layer F.Cu) (net 12))
@@
   (segment (start 93.98 99.06) (end 96.52 99.06) (width 0.5) (layer F.Cu) (net 19))
   (via (at 93.98 99.06) (size 1.5) (drill 0.8) (layers F.Cu B.Cu) (net 19))
+  (segment (start 68.58 111.76) (end 68.58 114.3) (width 0.5) (layer B.Cu) (net 33) (status 400000))
+  (via (at 68.58 114.3) (size 1.5) (drill 0.8) (layers F.Cu B.Cu) (net 33))
   (segment (start 68.58 111.76) (end 68.58 109.22) (width 0.5) (layer B.Cu) (net 33) (status C00000))
   (segment (start 66.04 116.84) (end 66.04 119.38) (width 0.5) (layer B.Cu) (net 34))
@@
   (segment (start 93.98 111.76) (end 93.98 114.3) (width 0.5) (layer B.Cu) (net 40))
   (segment (start 93.98 109.22) (end 93.98 111.76) (width 0.5) (layer B.Cu) (net 40) (status C00000))
+  (segment (start 106.68 99.06) (end 106.68 91.44) (width 0.5) (layer B.Cu) (net 41))
+  (via (at 106.68 91.44) (size 1.5) (drill 0.8) (layers F.Cu B.Cu) (net 41))
   (segment (start 109.219999 96.52) (end 109.22 99.06) (width 0.5) (layer B.Cu) (net 41) (status 400000))
   (segment (start 106.68 99.06) (end 106.68 101.6) (width 0.5) (layer B.Cu) (net 41) (status 800000))
